Commit message: xacro作成中

File: urdf/hekken.xacro (robot description, xacro)
@@ -91,10 +91,10 @@
     </xacro:macro>
     <xacro:macro name="asi_left" params="parent child xyz rpy">
-        <joint name="${child}_joint" type="revolute">
+        <joint name="${child}_joint" type="continuous">
             <origin xyz="${xyz}" rpy="${rpy}"/>
             <parent link="${parent}"/>
             <child link="${child}_link"/>
             <axis xyz="1 0 0"/>
-            <limit lower="${radians(-52)}" upper="${radians(38)}" effort="1.0" velocity="10.0"/>
+            <!--<limit lower="${radians(-52)}" upper="${radians(38)}" effort="1.0" velocity="10.0"/>-->
         </joint>
         <link name="${child}_link">
@@ -126,10 +126,10 @@
     </xacro:macro>
     <xacro:macro name="asi_right" params="parent child xyz rpy">
-        <joint name="${child}_joint" type="revolute">
+        <joint name="${child}_joint" type="continuous">
             <origin xyz="${xyz}" rpy="${rpy}"/>
             <parent link="${parent}"/>
             <child link="${child}_link"/>
             <axis xyz="1 0 0"/>
-            <limit lower="${radians(-52)}" upper="${radians(38)}" effort="1.0" velocity="10.0"/>
+            <!--<limit lower="${radians(-52)}" upper="${radians(38)}" effort="1.0" velocity="10.0"/>-->
         </joint>
         <link name="${child}_link">
@@ -157,4 +157,21 @@
             <gravity>true</gravity>
         </gazebo>
+    </xacro:macro>
+    <xacro:macro name="asi_secret_continuous" params="parent child xyz rpy">
+        <joint name="${child}_joint" type="continuous">
+            <origin xyz="${xyz}" rpy="${rpy}"/>
+            <parent link="${parent}"/>
+            <child link="${child}"/>
+            <axis xyz="1 0 0"/>
+        </joint>
+        <link name="${child}_link"/>
+    </xacro:macro>
+    <xacro:macro name="asi_secret_fixed" params="parent child xyz">
+        <joint name="${child}_joint" type="fixed">
+            <origin xyz="${xyz}" rpy="0 0 0"/>
+            <parent link="${parent}"/>
+            <child link="${child}"/>
+        </joint>
+        <link name="${child}_link"/>
     </xacro:macro>
     <link name="base_link"/>
@@ -195,4 +212,14 @@
     <xacro:asi_left parent="b_crank_link" child="b_asi_2" xyz="-0.033 0.0 -0.005" rpy="0 0 0"/>
     <xacro:asi_left parent="b_crank_link" child="b_asi_3" xyz="-0.051 ${-0.005*sin(radians(60))} ${-0.005*cos(radians(60))}" rpy="${radians(-37)} 0 0"/>
+    <xacro:asi_secret_continuous parent="b_asi_1_link" child="b_asi_1_secret1" xyz="0 0 0" rpy="0 0 0"/>
+    <xacro:asi_secret_continuous parent="b_asi_1_secret1_link" child="b_asi_1_secret2" xyz="0 0 0" rpy="0 0 0"/>
+    <xacro:asi_secret_fixed parent="b_asi_1_secret2_link" child="b_asi_1_base" xyz="0 0 0"/>
+    <xacro:asi_secret_fixed parent="body_link" child="b_1_mix" xyz="0 0 0"/>
+    <gazebo>
+        <joint name="b_asi_1_fix_joint">
+            <pose>0 0 0 0 0 0</pose>
+            <parent>
+        </joint>
+    </gazebo>
     <xacro:asi_left parent="c_crank_link" child="c_asi_1" xyz="-0.015 ${0.005*sin(radians(60))} ${-0.005*cos(radians(60))}" rpy="${radians(38)} 0 0"/>
     <xacro:asi_left parent="c_crank_link" child="c_asi_2" xyz="-0.033 0.0 -0.005" rpy="0 0 0"/>

Commit message: 座標計算中

File: urdf/hekken.xacro (robot description, xacro)
@@ -162,8 +162,9 @@
             <origin xyz="${xyz}" rpy="${rpy}"/>
             <parent link="${parent}"/>
-            <child link="${child}"/>
+            <child link="${child}_link"/>
             <axis xyz="1 0 0"/>
         </joint>
         <link name="${child}_link"/>
+        <gazebo reference="${child}_link"/>
     </xacro:macro>
     <xacro:macro name="asi_secret_fixed" params="parent child xyz">
@@ -171,7 +172,8 @@
             <origin xyz="${xyz}" rpy="0 0 0"/>
             <parent link="${parent}"/>
-            <child link="${child}"/>
+            <child link="${child}_link"/>
         </joint>
         <link name="${child}_link"/>
+        <gazebo reference="${child}_link"/>
     </xacro:macro>
     <link name="base_link"/>
@@ -212,5 +214,5 @@
     <xacro:asi_left parent="b_crank_link" child="b_asi_2" xyz="-0.033 0.0 -0.005" rpy="0 0 0"/>
     <xacro:asi_left parent="b_crank_link" child="b_asi_3" xyz="-0.051 ${-0.005*sin(radians(60))} ${-0.005*cos(radians(60))}" rpy="${radians(-37)} 0 0"/>
-    <xacro:asi_secret_continuous parent="b_asi_1_link" child="b_asi_1_secret1" xyz="0 0 0" rpy="0 0 0"/>
+    <xacro:asi_secret_continuous parent="b_asi_1_link" child="b_asi_1_secret1" xyz="0 ${(5*sqrt(3)/2)*0.001} ${((7.1*0.001)**2)-((5*sqrt(3)/2)*0.001)**2}" rpy="0 0 0"/>
     <xacro:asi_secret_continuous parent="b_asi_1_secret1_link" child="b_asi_1_secret2" xyz="0 0 0" rpy="0 0 0"/>
     <xacro:asi_secret_fixed parent="b_asi_1_secret2_link" child="b_asi_1_base" xyz="0 0 0"/>
@@ -219,5 +221,6 @@
         <joint name="b_asi_1_fix_joint">
             <pose>0 0 0 0 0 0</pose>
-            <parent>
+            <parent>b_1_mix_link</parent>
+            <child>b_asi_1_base_link</child>
         </joint>
     </gazebo>
