Commit message: 寸法指定完了

File: urdf/hekken.urdf (robot description, URDF)
Before this commit: robot hekken, 22 links, 21 joints
Joints:
- joint b_1_mix_joint: origin xyz=0 0 0 rpy=0 0 0 -> xyz=-0.1773 0.1225 0.013 rpy=0 0 0
- joint b_asi_1_base_joint: origin xyz=0 0 0 rpy=0 0 0 -> xyz=0 0.00788010753607 -0.00615661475326 rpy=0 0 0
- joint b_asi_1_secret1_joint: origin xyz=0 -0.00433012701892 3.166e-05 rpy=0 0 0 -> xyz=0 -7.25742165217e-05 0.00709962907363 rpy=0 0 0
- joint b_asi_1_secret2_joint: origin xyz=0 0 0 rpy=0 0 0 -> xyz=0 -0.0215007275907 0.0129278270823 rpy=0 0 0

File: urdf/hekken.xacro (robot description, xacro)
@@ -214,10 +214,14 @@
     <xacro:asi_left parent="b_crank_link" child="b_asi_2" xyz="-0.033 0.0 -0.005" rpy="0 0 0"/>
     <xacro:asi_left parent="b_crank_link" child="b_asi_3" xyz="-0.051 ${-0.005*sin(radians(60))} ${-0.005*cos(radians(60))}" rpy="${radians(-37)} 0 0"/>
-    <xacro:asi_secret_continuous parent="b_asi_1_link" child="b_asi_1_secret1" xyz="0 ${(5*sqrt(3)/2)*0.001} ${((7.1*0.001)**2)-((5*sqrt(3)/2)*0.001)**2}" rpy="0 0 0"/>
-    <xacro:asi_secret_continuous parent="b_asi_1_secret1_link" child="b_asi_1_secret2" xyz="0 0 0" rpy="0 0 0"/>
-    <xacro:asi_secret_fixed parent="b_asi_1_secret2_link" child="b_asi_1_base" xyz="0 0 0"/>
-    <xacro:asi_secret_fixed parent="body_link" child="b_1_mix" xyz="0 0 0"/>
+    <!--<xacro:asi_secret_continuous parent="b_asi_1_link" child="b_asi_1_secret1" xyz="0 ${-7.1*0.001*cos(radians(68)+(radians(60)-asin((5*sqrt(3))/(2*7.1))))} ${7.1*0.001*sin(radians(68)+(radians(60)-asin((5*sqrt(3))/(2*7.1))))}" rpy="0 0 0"/>-->
+    <xacro:asi_secret_continuous parent="b_asi_1_link" child="b_asi_1_secret1" xyz="0 ${-7.1*0.001*cos(radians(89.414328349))} ${7.1*0.001*sin(radians(89.414328349))}" rpy="0 0 0"/>
+    <!--<xacro:asi_secret_continuous parent="b_asi_1_secret1_link" child="b_asi_1_secret2" xyz="0 ${-((25*0.001*cos(radians(38)))+(5*0.001*cos(radians(68))-7.1*0.001*cos(radians(68)+(radians(60)-asin((5*sqrt(3))/(2*7.1))))))} ${-((sqrt(629.41)*0.001)**2-((25*0.001*cos(radians(38)))+(5*0.001*cos(radians(68))-7.1*0.001*cos(radians(68)+(radians(60)-asin((5*sqrt(3))/(2*7.1))))))**2)}" rpy="0 0 0"/>-->
+    <xacro:asi_secret_continuous parent="b_asi_1_secret1_link" child="b_asi_1_secret2" xyz="0 ${-0.001*sqrt(629.41)*cos(radians(31.017396292))} ${0.001*sqrt(629.41)*sin(radians(31.017396292))}" rpy="0 0 0"/>
+    <xacro:asi_secret_fixed parent="b_asi_1_secret2_link" child="b_asi_1_base" xyz="0 ${10*0.001*cos(radians(38))} ${-10*0.001*sin(radians(38))}"/>
+    <xacro:asi_secret_fixed parent="body_link" child="b_1_mix" xyz="${-0.1623-0.015} ${0.1375-0.015} 0.013"/>
     <gazebo>
-        <joint name="b_asi_1_fix_joint">
+        <joint name="b_asi_1_fix_joint" type="continuous">
+            <stopCfm>0.2</stopCfm>
+            <stopErp>0.2</stopErp>
             <pose>0 0 0 0 0 0</pose>
             <parent>b_1_mix_link</parent>

Commit message: gazeboでjointが表示されない

File: urdf/hekken.urdf (robot description, URDF)
Before this commit: robot hekken, 22 links, 21 joints
Joints:
- added joint b_asi_1_fix_joint: type continuous, parent b_1_mix_link, child b_asi_1_base_link, origin xyz=0 0 0 rpy=0 0 0, axis 1 0 0

File: urdf/hekken.xacro (robot description, xacro)
@@ -158,5 +158,5 @@
         </gazebo>
     </xacro:macro>
-    <xacro:macro name="asi_secret_continuous" params="parent child xyz rpy">
+    <xacro:macro name="asi_secret_continuous" params="parent child xyz rpy length">
         <joint name="${child}_joint" type="continuous">
             <origin xyz="${xyz}" rpy="${rpy}"/>
@@ -165,8 +165,22 @@
             <axis xyz="1 0 0"/>
         </joint>
-        <link name="${child}_link"/>
-        <gazebo reference="${child}_link"/>
-    </xacro:macro>
-    <xacro:macro name="asi_secret_fixed" params="parent child xyz">
+        <link name="${child}_link">
+            <collision>
+                <geometry>
+                    <cylinder radius="0.000001" length="0.000001"/>
+                </geometry>
+            </collision>
+            <inertial>
+                <origin xyz="0 0 0" rpy="0 0 0"/>
+                <mass value="0.000001"/>
+                <inertia ixx="0.1" ixy="0.1" ixz="0.1" iyy="0.1" iyz="0.1" izz="0.1"/>
+            </inertial>
+        </link>
+        <gazebo reference="${child}_link">
+            <material>Gazebo/Purple</material>
+            <gravity>false</gravity>
+        </gazebo>
+    </xacro:macro>
+    <xacro:macro name="asi_secret_fixed" params="parent child xyz length">
         <joint name="${child}_joint" type="fixed">
             <origin xyz="${xyz}" rpy="0 0 0"/>
@@ -174,5 +188,16 @@
             <child link="${child}_link"/>
         </joint>
-        <link name="${child}_link"/>
+        <link name="${child}_link">
+            <collision>
+                <geometry>
+                    <cylinder radius="0.000001" length="0.000001"/>
+                </geometry>
+            </collision>
+            <inertial>
+                <origin xyz="0 0 0" rpy="0 0 0"/>
+                <mass value="0.000001"/>
+                <inertia ixx="0.1" ixy="0.1" ixz="0.1" iyy="0.1" iyz="0.1" izz="0.1"/>
+            </inertial>
+        </link>
         <gazebo reference="${child}_link"/>
     </xacro:macro>
@@ -215,10 +240,15 @@
     <xacro:asi_left parent="b_crank_link" child="b_asi_3" xyz="-0.051 ${-0.005*sin(radians(60))} ${-0.005*cos(radians(60))}" rpy="${radians(-37)} 0 0"/>
     <!--<xacro:asi_secret_continuous parent="b_asi_1_link" child="b_asi_1_secret1" xyz="0 ${-7.1*0.001*cos(radians(68)+(radians(60)-asin((5*sqrt(3))/(2*7.1))))} ${7.1*0.001*sin(radians(68)+(radians(60)-asin((5*sqrt(3))/(2*7.1))))}" rpy="0 0 0"/>-->
-    <xacro:asi_secret_continuous parent="b_asi_1_link" child="b_asi_1_secret1" xyz="0 ${-7.1*0.001*cos(radians(89.414328349))} ${7.1*0.001*sin(radians(89.414328349))}" rpy="0 0 0"/>
+    <xacro:asi_secret_continuous parent="b_asi_1_link" child="b_asi_1_secret1" xyz="0 ${-7.1*0.001*cos(radians(89.414328349))} ${7.1*0.001*sin(radians(89.414328349))}" rpy="0 0 0" length="0.0071"/>
     <!--<xacro:asi_secret_continuous parent="b_asi_1_secret1_link" child="b_asi_1_secret2" xyz="0 ${-((25*0.001*cos(radians(38)))+(5*0.001*cos(radians(68))-7.1*0.001*cos(radians(68)+(radians(60)-asin((5*sqrt(3))/(2*7.1))))))} ${-((sqrt(629.41)*0.001)**2-((25*0.001*cos(radians(38)))+(5*0.001*cos(radians(68))-7.1*0.001*cos(radians(68)+(radians(60)-asin((5*sqrt(3))/(2*7.1))))))**2)}" rpy="0 0 0"/>-->
-    <xacro:asi_secret_continuous parent="b_asi_1_secret1_link" child="b_asi_1_secret2" xyz="0 ${-0.001*sqrt(629.41)*cos(radians(31.017396292))} ${0.001*sqrt(629.41)*sin(radians(31.017396292))}" rpy="0 0 0"/>
-    <xacro:asi_secret_fixed parent="b_asi_1_secret2_link" child="b_asi_1_base" xyz="0 ${10*0.001*cos(radians(38))} ${-10*0.001*sin(radians(38))}"/>
-    <xacro:asi_secret_fixed parent="body_link" child="b_1_mix" xyz="${-0.1623-0.015} ${0.1375-0.015} 0.013"/>
-    <gazebo>
+    <xacro:asi_secret_continuous parent="b_asi_1_secret1_link" child="b_asi_1_secret2" xyz="0 ${-0.001*sqrt(629.41)*cos(radians(31.017396292))} ${0.001*sqrt(629.41)*sin(radians(31.017396292))}" rpy="0 0 0" length="${sqrt(629.41)*0.001}"/>
+    <xacro:asi_secret_fixed parent="b_asi_1_secret2_link" child="b_asi_1_base" xyz="0 ${10*0.001*cos(radians(38))} ${-10*0.001*sin(radians(38))}" length="0.01"/>
+    <xacro:asi_secret_fixed parent="body_link" child="b_1_mix" xyz="${-0.1623-0.015} ${0.1375-0.015} 0.013" length="0.1"/>
+    <!--<joint name="b_asi_1_fix_joint" type="fixed">
+        <origin xyz="0 0 0" rpy="0 0 0"/>
+        <parent link="b_1_mix_link"/>
+        <child link="b_asi_1_base_link"/>
+    </joint>-->
+    <!--<gazebo>
         <joint name="b_asi_1_fix_joint" type="continuous">
             <stopCfm>0.2</stopCfm>
@@ -228,5 +258,5 @@
             <child>b_asi_1_base_link</child>
         </joint>
-    </gazebo>
+    </gazebo>-->
     <xacro:asi_left parent="c_crank_link" child="c_asi_1" xyz="-0.015 ${0.005*sin(radians(60))} ${-0.005*cos(radians(60))}" rpy="${radians(38)} 0 0"/>
     <xacro:asi_left parent="c_crank_link" child="c_asi_2" xyz="-0.033 0.0 -0.005" rpy="0 0 0"/>
